File: kicad/pcb_main_r2/mintypcb.kicad_pcb (KiCad board)
At the start: 2 copper layers, 89 x 55.5 mm, 158 parts, among them J101 USB_C_Receptacle_USB2.0_14P, J102 S2B-PH-SM4-TB, J103 FPC09-Q1.0-8, J106 Conn_02x15_Odd_Even, J107 Conn_02x15_Odd_Even, J108 Conn_02x15_Odd_Even, Q101 3415, Q102 3415, Q103 BSS138, SW101 SKQGABE010, SW102 SKRRAAE010, SW103 SKQGABE010, SW104 SKRRAAE010, SW105 SKQGABE010, SW106 SKRRAAE010, SW107 see note 1, SW108 SKRRAAE010, SW109 see note 1, SW110 SKRRAAE010, SW111 see note 1, SW112 SKRRAAE010, SW113 see note 1, SW114 SKRRAAE010, SW115 SKQGABE010, SW116 SKRRAAE010, U101 LMV393, U102 MCP73833T-FCI/MF, U103 PAM2401SCADJ, U104 MAX98357A, U106 74AHCT1G125, U107 USBLC6-2SC6

Commit message: added sofware controls
Parts:
- renumbered D7 to D1, D6 to D10, D8 to D2, D9 to D3, D10 to D4, D1 to D5, D2 to D6, D3 to D7, D4 to D8, D5 to D9
Changed lines of the file:
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@@
 		(descr "2.0mm x 2.0mm Addressable RGB LED NeoPixel Nano, 12 mA, https://cdn-shop.adafruit.com/product-files/4684/4684_WS2812B-2020_V1.3_EN.pdf")
 		(tags "LED RGB NeoPixel Nano PLCC-4 2020")
-		(property "Reference" "D5"
+		(property "Reference" "D9"
 			(at 0 -2.000001 225)
 			(layer "F.SilkS")
@@
 			(size 0.7 0.7)
 			(layers "F.Cu" "F.Mask" "F.Paste")
-			(net "Net-(D5-DOUT)")
+			(net "Net-(D10-DIN)")
 			(pinfunction "DOUT_1")
 			(pintype "output")
@@
 			(size 0.7 0.7)
 			(layers "F.Cu" "F.Mask" "F.Paste")
-			(net "Net-(D4-DOUT)")
+			(net "Net-(D8-DOUT)")
 			(pinfunction "DIN_3")
 			(pintype "input")
@@
 		(descr "2.0mm x 2.0mm Addressable RGB LED NeoPixel Nano, 12 mA, https://cdn-shop.adafruit.com/product-files/4684/4684_WS2812B-2020_V1.3_EN.pdf")
 		(tags "LED RGB NeoPixel Nano PLCC-4 2020")
-		(property "Reference" "D3"
+		(property "Reference" "D7"
 			(at 0 -2.000001 45)
 			(layer "F.SilkS")
@@
 			(size 0.7 0.7)
 			(layers "F.Cu" "F.Mask" "F.Paste")
-			(net "Net-(D3-DOUT)")
+			(net "Net-(D7-DOUT)")
 			(pinfunction "DOUT_1")
 			(pintype "output")
@@
 			(size 0.7 0.7)
 			(layers "F.Cu" "F.Mask" "F.Paste")
-			(net "Net-(D2-DOUT)")
+			(net "Net-(D6-DOUT)")
 			(pinfunction "DIN_3")
 			(pintype "input")
@@
 		(descr "2.0mm x 2.0mm Addressable RGB LED NeoPixel Nano, 12 mA, https://cdn-shop.adafruit.com/product-files/4684/4684_WS2812B-2020_V1.3_EN.pdf")
 		(tags "LED RGB NeoPixel Nano PLCC-4 2020")
-		(property "Reference" "D1"
+		(property "Reference" "D5"
 			(at 0 -2.000001 0)
 			(layer "F.SilkS")
@@
 			(size 0.7 0.7)
 			(layers "F.Cu" "F.Mask" "F.Paste")
-			(net "Net-(D1-DOUT)")
+			(net "Net-(D5-DOUT)")
 			(pinfunction "DOUT_1")
 			(pintype "output")
@@
 		(descr "2.0mm x 2.0mm Addressable RGB LED NeoPixel Nano, 12 mA, https://cdn-shop.adafruit.com/product-files/4684/4684_WS2812B-2020_V1.3_EN.pdf")
 		(tags "LED RGB NeoPixel Nano PLCC-4 2020")
-		(property "Reference" "D6"
+		(property "Reference" "D10"
 			(at 0 -2.000001 135)
 			(layer "F.SilkS")
@@
 			(size 0.7 0.7)
 			(layers "F.Cu" "F.Mask" "F.Paste")
-			(net "unconnected-(D6-DOUT-Pad1)")
+			(net "unconnected-(D10-DOUT-Pad1)")
 			(pinfunction "DOUT_1")
 			(pintype "output")
@@
 			(size 0.7 0.7)
 			(layers "F.Cu" "F.Mask" "F.Paste")
-			(net "Net-(D5-DOUT)")
+			(net "Net-(D10-DIN)")
 			(pinfunction "DIN_3")
 			(pintype "input")
@@
 		(descr "2.0mm x 2.0mm Addressable RGB LED NeoPixel Nano, 12 mA, https://cdn-shop.adafruit.com/product-files/4684/4684_WS2812B-2020_V1.3_EN.pdf")
 		(tags "LED RGB NeoPixel Nano PLCC-4 2020")
-		(property "Reference" "D10"
+		(property "Reference" "D4"
 			(at 0 -2.000001 315)
 			(layer "F.SilkS")
@@
 			(size 0.7 0.7)
 			(layers "F.Cu" "F.Mask" "F.Paste")
-			(net "Net-(D10-DIN)")
+			(net "Net-(D3-DOUT)")
 			(pinfunction "DIN_3")
 			(pintype "input")
@@
 		(descr "2.0mm x 2.0mm Addressable RGB LED NeoPixel Nano, 12 mA, https://cdn-shop.adafruit.com/product-files/4684/4684_WS2812B-2020_V1.3_EN.pdf")
 		(tags "LED RGB NeoPixel Nano PLCC-4 2020")
-		(property "Reference" "D8"
+		(property "Reference" "D2"
 			(at 0 -2.000001 135)
 			(layer "F.SilkS")
@@
 			(size 0.7 0.7)
 			(layers "F.Cu" "F.Mask" "F.Paste")
-			(net "Net-(D8-DOUT)")
+			(net "Net-(D2-DOUT)")
 			(pinfunction "DOUT_1")
 			(pintype "output")
@@
 			(size 0.7 0.7)
 			(layers "F.Cu" "F.Mask" "F.Paste")
-			(net "Net-(D7-DOUT)")
+			(net "Net-(D1-DOUT)")
 			(pinfunction "DIN_3")
 			(pintype "input")
@@
 		(descr "2.0mm x 2.0mm Addressable RGB LED NeoPixel Nano, 12 mA, https://cdn-shop.adafruit.com/product-files/4684/4684_WS2812B-2020_V1.3_EN.pdf")
 		(tags "LED RGB NeoPixel Nano PLCC-4 2020")
-		(property "Reference" "D9"
+		(property "Reference" "D3"
 			(at 0 -2.000001 45)
 			(layer "F.SilkS")
@@
 			(size 0.7 0.7)
 			(layers "F.Cu" "F.Mask" "F.Paste")
-			(net "Net-(D10-DIN)")
+			(net "Net-(D3-DOUT)")
 			(pinfunction "DOUT_1")
 			(pintype "output")
@@
 			(size 0.7 0.7)
 			(layers "F.Cu" "F.Mask" "F.Paste")
-			(net "Net-(D8-DOUT)")
+			(net "Net-(D2-DOUT)")
 			(pinfunction "DIN_3")
 			(pintype "input")
@@
 		(descr "2.0mm x 2.0mm Addressable RGB LED NeoPixel Nano, 12 mA, https://cdn-shop.adafruit.com/product-files/4684/4684_WS2812B-2020_V1.3_EN.pdf")
 		(tags "LED RGB NeoPixel Nano PLCC-4 2020")
-		(property "Reference" "D4"
+		(property "Reference" "D8"
 			(at 0 -2.000001 315)
 			(layer "F.SilkS")
@@
 			(size 0.7 0.7)
 			(layers "F.Cu" "F.Mask" "F.Paste")
-			(net "Net-(D4-DOUT)")
+			(net "Net-(D8-DOUT)")
 			(pinfunction "DOUT_1")
 			(pintype "output")
@@
 			(size 0.7 0.7)
 			(layers "F.Cu" "F.Mask" "F.Paste")
-			(net "Net-(D3-DOUT)")
+			(net "Net-(D7-DOUT)")
 			(pinfunction "DIN_3")
 			(pintype "input")
@@
 		(descr "2.0mm x 2.0mm Addressable RGB LED NeoPixel Nano, 12 mA, https://cdn-shop.adafruit.com/product-files/4684/4684_WS2812B-2020_V1.3_EN.pdf")
 		(tags "LED RGB NeoPixel Nano PLCC-4 2020")
-		(property "Reference" "D2"
+		(property "Reference" "D6"
 			(at 0 -2.000001 0)
 			(layer "F.SilkS")
@@
 			(size 0.7 0.7)
 			(layers "F.Cu" "F.Mask" "F.Paste")
-			(net "Net-(D2-DOUT)")
+			(net "Net-(D6-DOUT)")
 			(pinfunction "DOUT_1")
 			(pintype "output")
@@
 			(size 0.7 0.7)
 			(layers "F.Cu" "F.Mask" "F.Paste")
-			(net "Net-(D1-DOUT)")
+			(net "Net-(D5-DOUT)")
 			(pinfunction "DIN_3")
 			(pintype "input")
@@
 		(descr "2.0mm x 2.0mm Addressable RGB LED NeoPixel Nano, 12 mA, https://cdn-shop.adafruit.com/product-files/4684/4684_WS2812B-2020_V1.3_EN.pdf")
 		(tags "LED RGB NeoPixel Nano PLCC-4 2020")
-		(property "Reference" "D7"
+		(property "Reference" "D1"
 			(at 0 -2.000001 225)
 			(layer "F.SilkS")
@@
 			(size 0.7 0.7)
 			(layers "F.Cu" "F.Mask" "F.Paste")
-			(net "Net-(D7-DOUT)")
+			(net "Net-(D1-DOUT)")
 			(pinfunction "DOUT_1")
 			(pintype "output")
@@
 		(width 0.2)
 		(layer "F.Cu")
-		(net "Net-(D5-DOUT)")
+		(net "Net-(D10-DIN)")
 	)
 	(segment
@@
 		(width 0.2)
 		(layer "F.Cu")
-		(net "Net-(D5-DOUT)")
+		(net "Net-(D10-DIN)")
 	)
 	(segment
@@
 		(width 0.2)
 		(layer "F.Cu")
-		(net "Net-(D5-DOUT)")
+		(net "Net-(D10-DIN)")
 	)
 	(segment
@@
 		(width 0.2)
 		(layer "F.Cu")
-		(net "Net-(D4-DOUT)")
+		(net "Net-(D8-DOUT)")
 	)
 	(segment
@@
 		(width 0.2)
 		(layer "F.Cu")
-		(net "Net-(D4-DOUT)")
+		(net "Net-(D8-DOUT)")
 	)
 	(segment
@@
 		(width 0.2)
 		(layer "F.Cu")
-		(net "Net-(D4-DOUT)")
+		(net "Net-(D8-DOUT)")
 	)
 	(segment
@@
 		(width 0.2)
 		(layer "F.Cu")
-		(net "Net-(D4-DOUT)")
+		(net "Net-(D8-DOUT)")
 	)
 	(via
@@
 		(drill 0.3)
 		(layers "F.Cu" "B.Cu")
-		(net "Net-(D4-DOUT)")
+		(net "Net-(D8-DOUT)")
 	)
 	(via
@@
 		(drill 0.3)
 		(layers "F.Cu" "B.Cu")
-		(net "Net-(D4-DOUT)")
+		(net "Net-(D8-DOUT)")
 	)
 	(segment
@@
 		(width 0.2)
 		(layer "B.Cu")
-		(net "Net-(D4-DOUT)")
+		(net "Net-(D8-DOUT)")
 	)
 	(segment
@@
 		(width 0.2)
 		(layer "F.Cu")
-		(net "Net-(D3-DOUT)")
+		(net "Net-(D7-DOUT)")
 	)
 	(segment
@@
 		(width 0.2)
 		(layer "F.Cu")
-		(net "Net-(D3-DOUT)")
+		(net "Net-(D7-DOUT)")
 	)
 	(segment
@@
 		(width 0.2)
 		(layer "F.Cu")
-		(net "Net-(D3-DOUT)")
+		(net "Net-(D7-DOUT)")
 	)
 	(segment
@@
 		(width 0.2)
 		(layer "F.Cu")
-		(net "Net-(D3-DOUT)")
+		(net "Net-(D7-DOUT)")
 	)
 	(segment
@@
 		(width 0.2)
 		(layer "F.Cu")
-		(net "Net-(D3-DOUT)")
+		(net "Net-(D7-DOUT)")
 	)
 	(segment
@@
 		(width 0.2)
 		(layer "F.Cu")
-		(net "Net-(D3-DOUT)")
+		(net "Net-(D7-DOUT)")
 	)
 	(segment
@@
 		(width 0.2)
 		(layer "F.Cu")
-		(net "Net-(D3-DOUT)")
+		(net "Net-(D7-DOUT)")
 	)
 	(segment
@@
 		(width 0.2)
 		(layer "F.Cu")
-		(net "Net-(D2-DOUT)")
+		(net "Net-(D6-DOUT)")
 	)
 	(segment
@@
 		(width 0.2)
 		(layer "F.Cu")
-		(net "Net-(D2-DOUT)")
+		(net "Net-(D6-DOUT)")
 	)
 	(segment
@@
 		(width 0.2)
 		(layer "F.Cu")
-		(net "Net-(D2-DOUT)")
+		(net "Net-(D6-DOUT)")
 	)
 	(segment
@@
 		(width 0.2)
 		(layer "F.Cu")
-		(net "Net-(D2-DOUT)")
+		(net "Net-(D6-DOUT)")
 	)
 	(segment
@@
 		(width 0.2)
 		(layer "F.Cu")
-		(net "Net-(D1-DOUT)")
+		(net "Net-(D5-DOUT)")
 	)
 	(segment
@@
 		(width 0.2)
 		(layer "F.Cu")
-		(net "Net-(D1-DOUT)")
+		(net "Net-(D5-DOUT)")
 	)
 	(segment
@@
 		(width 0.2)
 		(layer "F.Cu")
-		(net "Net-(D1-DOUT)")
+		(net "Net-(D5-DOUT)")
 	)
 	(segment
@@
 		(width 0.2)
 		(layer "F.Cu")
-		(net "Net-(D10-DIN)")
+		(net "Net-(D3-DOUT)")
 	)
 	(segment
@@
 		(width 0.2)
 		(layer "F.Cu")
-		(net "Net-(D10-DIN)")
+		(net "Net-(D3-DOUT)")
 	)
 	(segment
@@
 		(width 0.2)
 		(layer "F.Cu")
-		(net "Net-(D10-DIN)")
+		(net "Net-(D3-DOUT)")
 	)
 	(segment
@@
 		(width 0.2)
 		(layer "F.Cu")
-		(net "Net-(D10-DIN)")
+		(net "Net-(D3-DOUT)")
 	)
 	(segment
@@
 		(width 0.2)
 		(layer "F.Cu")
-		(net "Net-(D10-DIN)")
+		(net "Net-(D3-DOUT)")
 	)
 	(segment
@@
 		(width 0.2)
 		(layer "F.Cu")
-		(net "Net-(D10-DIN)")
+		(net "Net-(D3-DOUT)")
 	)
 	(segment
@@
 		(width 0.2)
 		(layer "F.Cu")
-		(net "Net-(D10-DIN)")
+		(net "Net-(D3-DOUT)")
 	)
 	(segment
@@
 		(width 0.2)
 		(layer "F.Cu")
-		(net "Net-(D8-DOUT)")
+		(net "Net-(D2-DOUT)")
 	)
 	(segment
@@
 		(width 0.2)
 		(layer "F.Cu")
-		(net "Net-(D8-DOUT)")
+		(net "Net-(D2-DOUT)")
 	)
 	(segment
@@
 		(width 0.2)
 		(layer "F.Cu")
-		(net "Net-(D8-DOUT)")
+		(net "Net-(D2-DOUT)")
 	)
 	(segment
@@
 		(width 0.2)
 		(layer "F.Cu")
-		(net "Net-(D8-DOUT)")
+		(net "Net-(D2-DOUT)")
 	)
 	(segment
@@
 		(width 0.2)
 		(layer "F.Cu")
-		(net "Net-(D7-DOUT)")
+		(net "Net-(D1-DOUT)")
 	)
 	(segment
@@
 		(width 0.2)
 		(layer "F.Cu")
-		(net "Net-(D7-DOUT)")
+		(net "Net-(D1-DOUT)")
 	)
 	(segment
@@
 		(width 0.2)
 		(layer "F.Cu")
-		(net "Net-(D7-DOUT)")
+		(net "Net-(D1-DOUT)")
 	)
 	(segment
@@
 		(width 0.2)
 		(layer "F.Cu")
-		(net "Net-(D7-DOUT)")
+		(net "Net-(D1-DOUT)")
 	)
 	(segment
@@
 		(width 0.2)
 		(layer "F.Cu")
-		(net "Net-(D7-DOUT)")
+		(net "Net-(D1-DOUT)")
 	)
 	(segment
@@
 		(width 0.2)
 		(layer "F.Cu")
-		(net "Net-(D7-DOUT)")
+		(net "Net-(D1-DOUT)")
 	)
 	(segment
