File: kicad/pcb_main_r2/mintypcb.kicad_sch (KiCad schematic)
At the start: 155 parts, among them J101 USB_C_Receptacle_USB2.0_14P, J102 S2B-PH-SM4-TB, J103 FPC09-Q1.0-8, J106 Conn_02x15_Odd_Even, J107 Conn_02x15_Odd_Even, J108 Conn_02x15_Odd_Even, Q101 3415, Q102 3415, Q103 BSS138, SW101 SKQGABE010, SW102 SKRRAAE010, SW103 SKQGABE010, SW104 SKRRAAE010, SW105 SKQGABE010, SW106 SKRRAAE010, SW107 see note 1, SW108 SKRRAAE010, SW109 see note 1, SW110 SKRRAAE010, SW111 see note 1, SW112 SKRRAAE010, SW113 see note 1, SW114 SKRRAAE010, SW115 SKQGABE010, SW116 SKRRAAE010, U101 LMV393, U102 MCP73833T-FCI/MF, U103 PAM2401SCADJ, U104 MAX98357A, U106 74AHCT1G125, U107 USBLC6-2SC6

Commit message: changed display brightness control port
Connections:
- net RST: now also A101.16 (GEN4/GPIO23), TP112.1; no longer A101.18 (GEN5/GPIO24), TP114.1
- net UP: now also A101.18 (GEN5/GPIO24), TP114.1; no longer A101.16 (GEN4/GPIO23), TP112.1
Changed lines of the file:
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@@
 		)
 	)
-	(label "RST"
+	(label "UP"
 		(at 88.9 161.29 0)
 		(effects
@@
 		)
 	)
-	(label "UP"
+	(label "RST"
 		(at 88.9 158.75 0)
 		(effects

Commit message: added sofware controls
Parts:
- renumbered D7 to D1, D6 to D10, D8 to D2, D9 to D3, D10 to D4, D1 to D5, D2 to D6, D3 to D7, D4 to D8, D5 to D9
Changed lines of the file:
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@@
 		(in_pos_files yes)
 		(dnp no)
-		(property "Reference" "D7"
+		(property "Reference" "D1"
 			(at 153.162 263.398 0)
 			(show_name no)
@@
 			(project "mintypcb"
 				(path "/c809f0b5-674b-425f-afd3-ebaa2d8ff300"
-					(reference "D7")
+					(reference "D1")
 					(unit 1)
 				)
@@
 		(in_pos_files yes)
 		(dnp no)
-		(property "Reference" "D3"
+		(property "Reference" "D7"
 			(at 173.482 232.918 0)
 			(show_name no)
@@
 			(project "mintypcb"
 				(path "/c809f0b5-674b-425f-afd3-ebaa2d8ff300"
-					(reference "D3")
+					(reference "D7")
 					(unit 1)
 				)
@@
 		(in_pos_files yes)
 		(dnp no)
-		(property "Reference" "D2"
+		(property "Reference" "D6"
 			(at 153.162 232.918 0)
 			(show_name no)
@@
 			(project "mintypcb"
 				(path "/c809f0b5-674b-425f-afd3-ebaa2d8ff300"
-					(reference "D2")
+					(reference "D6")
 					(unit 1)
 				)
@@
 		(in_pos_files yes)
 		(dnp no)
-		(property "Reference" "D6"
+		(property "Reference" "D10"
 			(at 132.842 263.398 0)
 			(show_name no)
@@
 			(project "mintypcb"
 				(path "/c809f0b5-674b-425f-afd3-ebaa2d8ff300"
-					(reference "D6")
+					(reference "D10")
 					(unit 1)
 				)
@@
 		(in_pos_files yes)
 		(dnp no)
-		(property "Reference" "D1"
+		(property "Reference" "D5"
 			(at 132.842 232.918 0)
 			(show_name no)
@@
 			(project "mintypcb"
 				(path "/c809f0b5-674b-425f-afd3-ebaa2d8ff300"
-					(reference "D1")
+					(reference "D5")
 					(unit 1)
 				)
@@
 		(in_pos_files yes)
 		(dnp no)
-		(property "Reference" "D5"
+		(property "Reference" "D9"
 			(at 214.122 232.918 0)
 			(show_name no)
@@
 			(project "mintypcb"
 				(path "/c809f0b5-674b-425f-afd3-ebaa2d8ff300"
-					(reference "D5")
+					(reference "D9")
 					(unit 1)
 				)
@@
 		(in_pos_files yes)
 		(dnp no)
-		(property "Reference" "D9"
+		(property "Reference" "D3"
 			(at 193.802 263.398 0)
 			(show_name no)
@@
 			(project "mintypcb"
 				(path "/c809f0b5-674b-425f-afd3-ebaa2d8ff300"
-					(reference "D9")
+					(reference "D3")
 					(unit 1)
 				)
@@
 		(in_pos_files yes)
 		(dnp no)
-		(property "Reference" "D4"
+		(property "Reference" "D8"
 			(at 193.802 232.918 0)
 			(show_name no)
@@
 			(project "mintypcb"
 				(path "/c809f0b5-674b-425f-afd3-ebaa2d8ff300"
-					(reference "D4")
+					(reference "D8")
 					(unit 1)
 				)
@@
 		(in_pos_files yes)
 		(dnp no)
-		(property "Reference" "D8"
+		(property "Reference" "D2"
 			(at 173.482 263.398 0)
 			(show_name no)
@@
 			(project "mintypcb"
 				(path "/c809f0b5-674b-425f-afd3-ebaa2d8ff300"
-					(reference "D8")
+					(reference "D2")
 					(unit 1)
 				)
@@
 		(in_pos_files yes)
 		(dnp no)
-		(property "Reference" "D10"
+		(property "Reference" "D4"
 			(at 214.122 263.398 0)
 			(show_name no)
@@
 			(project "mintypcb"
 				(path "/c809f0b5-674b-425f-afd3-ebaa2d8ff300"
-					(reference "D10")
+					(reference "D4")
 					(unit 1)
 				)
